File: driver-board/driver-board.kicad_sch (KiCad schematic)
At the start: 14 parts, among them J9 Conn_01x06, Q10 Q_NPN_BEC, Q9 Q_NPN_BEC, SW1 222AMVBAR, U4 ESP32-C3-WROOM-02-N4

Commit message: schematic updates for r1
Parts:
- added J12: Conn_01x02, Connector_Phoenix_MC:PhoenixContact_MCV_1,5_2-GF-3.81_1x02_P3.81mm_Vertical_ThreadedFlange_MountHole, symbol Connector_Generic:Conn_01x02
- added R27, R28: 10k, Resistor_SMD:R_0805_2012Metric, symbol Device:R_Small_US
Connections:
- net +3.3V: now also R27.2, R28.2
- net GND: now also J12.2 (Pin_2)
- net c6: now also U4.13 (IO18); no longer U4.7 (IO8)
- net at U4.14 (IO19): now also J12.1 (Pin_1), R28.1
- new net: R27.1, U4.7 (IO8)
