File: driver-board/driver0.kicad_sch (KiCad schematic)
At the start: 5 parts, among them J1 Conn_01x02, Q1 BUK7880-55A

Commit message: new board
Parts:
- removed Q1: BUK7880-55A, Package_TO_SOT_SMD:SOT-223-3_TabPin2, symbol Transistor_FET:BUK7880-55A
- added Q11: ZXM61N03FTA, Package_TO_SOT_SMD:SOT-23-3, symbol Transistor_FET:Q_NMOS_GSD
- R1: value 4.7k -> 0
Connections:
- net GND: now also Q11.2 (S)
- net at R1.2, R2.2: now also Q11.1 (G)
- net at D1.2 (A), J1.2 (Pin_2): now also Q11.3 (D)
Changed lines of the file:
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@@
-	)
-	(symbol
-		(lib_id "Transistor_FET:BUK7880-55A")
-		(at 165.1 92.71 0)
-		(unit 1)
-		(exclude_from_sim no)
-		(in_bom yes)
-		(on_board yes)
-		(dnp no)
-		(fields_autoplaced yes)
-		(property "Reference" "Q1"
-			(at 170.307 91.4978 0)
-			(effects
-				(font
-					(size 1.27 1.27)
-				)
-				(justify left)
-			)
-		)
-		(property "Value" "BUK7880-55A"
-			(at 170.307 93.9221 0)
-			(effects
-				(font
-					(size 1.27 1.27)
-				)
-				(justify left)
-			)
-		)
-		(property "Footprint" "Package_TO_SOT_SMD:SOT-223-3_TabPin2"
-			(at 170.18 94.615 0)
-			(effects
-				(font
-					(size 1.27 1.27)
-					(italic yes)
-				)
-				(justify left)
-				(hide yes)
-			)
-		)
-		(property "Datasheet" "https://assets.nexperia.com/documents/data-sheet/BUK7880-55A.pdf"
-			(at 170.18 96.52 0)
-			(effects
-				(font
-					(size 1.27 1.27)
-				)
-				(justify left)
-				(hide yes)
-			)
-		)
-		(property "Description" "7A Id, 55V Vds, N-Channel Enhancement Mode MOSFET, SOT-223"
-			(at 165.1 92.71 0)
-			(effects
-				(font
-					(size 1.27 1.27)
-				)
-				(hide yes)
-			)
-		)
-		(pin "2"
-		)
-		(pin "1"
-		)
-		(pin "3"
-		)
-		(instances
-			(project "driver-board"
-				(path "/3e314726-7059-4cf1-a457-28a818b66c88/119ff494-b194-43eb-83d5-0f887251f180"
-					(reference "Q6")
-					(unit 1)
-				)
-				(path "/3e314726-7059-4cf1-a457-28a818b66c88/7d631dd7-8150-4150-b9ae-ac3cc1de9e4f"
-					(reference "Q5")
-					(unit 1)
-				)
-				(path "/3e314726-7059-4cf1-a457-28a818b66c88/7fb9460a-2591-4e13-bcf7-abe67859cef0"
-					(reference "Q8")
-					(unit 1)
-				)
-				(path "/3e314726-7059-4cf1-a457-28a818b66c88/b1385036-17e2-455d-858c-2a9ed54f1ad3"
-					(reference "Q3")
-					(unit 1)
-				)
-				(path "/3e314726-7059-4cf1-a457-28a818b66c88/b4181847-7a43-4500-bd8e-7b5693dc7546"
-					(reference "Q1")
-					(unit 1)
-				)
-				(path "/3e314726-7059-4cf1-a457-28a818b66c88/b5934f9c-5359-4230-944d-cb36da629d67"
-					(reference "Q7")
-					(unit 1)
-				)
-				(path "/3e314726-7059-4cf1-a457-28a818b66c88/ca198ab4-2dfe-4f1b-aeb4-730993e48968"
-					(reference "Q2")
-					(unit 1)
-				)
-				(path "/3e314726-7059-4cf1-a457-28a818b66c88/ec1069f6-7b9e-4d48-bdab-0db2689c016a"
-					(reference "Q4")
-					(unit 1)
-				)
-			)
-		)
 	)
 	(symbol
@@
 	)
 	(symbol
+		(lib_id "Transistor_FET:Q_NMOS_GSD")
+		(at 165.1 92.71 0)
+		(unit 1)
+		(exclude_from_sim no)
+		(in_bom yes)
+		(on_board yes)
+		(dnp no)
+		(fields_autoplaced yes)
+		(property "Reference" "Q11"
+			(at 170.307 91.4978 0)
+			(effects
+				(font
+					(size 1.27 1.27)
+				)
+				(justify left)
+			)
+		)
+		(property "Value" "ZXM61N03FTA"
+			(at 170.307 93.9221 0)
+			(effects
+				(font
+					(size 1.27 1.27)
+				)
+				(justify left)
+			)
+		)
+		(property "Footprint" "Package_TO_SOT_SMD:SOT-23-3"
+			(at 170.18 90.17 0)
+			(effects
+				(font
+					(size 1.27 1.27)
+				)
+				(hide yes)
+			)
+		)
+		(property "Datasheet" "~"
+			(at 165.1 92.71 0)
+			(effects
+				(font
+					(size 1.27 1.27)
+				)
+				(hide yes)
+			)
+		)
+		(property "Description" "N-MOSFET transistor, gate/source/drain"
+			(at 165.1 92.71 0)
+			(effects
+				(font
+					(size 1.27 1.27)
+				)
+				(hide yes)
+			)
+		)
+		(pin "2"
+		)
+		(pin "3"
+		)
+		(pin "1"
+		)
+		(instances
+			(project ""
+				(path "/3e314726-7059-4cf1-a457-28a818b66c88/119ff494-b194-43eb-83d5-0f887251f180"
+					(reference "Q16")
+					(unit 1)
+				)
+				(path "/3e314726-7059-4cf1-a457-28a818b66c88/7d631dd7-8150-4150-b9ae-ac3cc1de9e4f"
+					(reference "Q15")
+					(unit 1)
+				)
+				(path "/3e314726-7059-4cf1-a457-28a818b66c88/7fb9460a-2591-4e13-bcf7-abe67859cef0"
+					(reference "Q18")
+					(unit 1)
+				)
+				(path "/3e314726-7059-4cf1-a457-28a818b66c88/b1385036-17e2-455d-858c-2a9ed54f1ad3"
+					(reference "Q13")
+					(unit 1)
+				)
+				(path "/3e314726-7059-4cf1-a457-28a818b66c88/b4181847-7a43-4500-bd8e-7b5693dc7546"
+					(reference "Q11")
+					(unit 1)
+				)
+				(path "/3e314726-7059-4cf1-a457-28a818b66c88/b5934f9c-5359-4230-944d-cb36da629d67"
+					(reference "Q17")
+					(unit 1)
+				)
+				(path "/3e314726-7059-4cf1-a457-28a818b66c88/ca198ab4-2dfe-4f1b-aeb4-730993e48968"
+					(reference "Q12")
+					(unit 1)
+				)
+				(path "/3e314726-7059-4cf1-a457-28a818b66c88/ec1069f6-7b9e-4d48-bdab-0db2689c016a"
+					(reference "Q14")
+					(unit 1)
+				)
+			)
+		)
+	)
+	(symbol
 		(lib_id "power:+12V")
 		(at 167.64 66.04 0)
@@
 			)
 		)
-		(property "Value" "4.7k"
+		(property "Value" "0"
 			(at 143.51 90.1008 90)
 			(effects
